Commit message: Chay map cung ko xong! Ga

File: src/agv_gazebo/xacro_agv/agv_urdf.xacro (robot description, xacro)
@@ -100,5 +100,5 @@
           <publishWheelTF>false</publishWheelTF>
           <!-- Set to true to publish transforms for the odometry, defaults to true -->
-          <publishOdom>false</publishOdom>
+          <publishOdom>true</publishOdom>
           <!-- Set to true to publish sensor_msgs/JointState on /joint_states for the wheel joints, defaults to false -->
           <publishWheelJointState>true</publishWheelJointState>

File: src/agv_urdf/urdf/agv_urdf.urdf (robot description, URDF)
Before this commit: robot agv_urdf, 8 links, 7 joints
Joints:
- joint MT_behind_left_jt: origin xyz=-0.10998 0.095 -0.019 rpy=0 0 0 -> xyz=-0.10998 0.095 -0.029 rpy=0 0 0
- joint MT_behind_right_jt: origin xyz=-0.10998 -0.095 -0.019 rpy=0 0 0 -> xyz=-0.10998 -0.095 -0.029 rpy=0 0 0
- joint MT_up_left_jt: origin xyz=0.11002 0.095 -0.019 rpy=0 0 0 -> xyz=0.11002 0.095 -0.029 rpy=0 0 0
- joint MT_up_right_jt: origin xyz=0.11002 -0.095 -0.019 rpy=0 0 0 -> xyz=0.11002 -0.095 -0.029 rpy=0 0 0
