Commit message: half a goal

File: src/agv_gazebo/xacro_agv/caster_behind_left.xacro (robot description, xacro)
@@ -25,5 +25,5 @@
     </link>
     <joint name="MT_behind_left_jt" type="fixed">
-      <origin xyz="-0.10998 0.095 -0.019" rpy="0 0 0" />
+      <origin xyz="-0.10998 0.095 -0.0204" rpy="0 0 0" />
       <parent link="base_link" />
       <child link="MT_behind_left" />

File: src/agv_gazebo/xacro_agv/caster_behind_right.xacro (robot description, xacro)
@@ -25,5 +25,5 @@
     </link>
     <joint name="MT_behind_right_jt" type="fixed">
-      <origin xyz="-0.10998 -0.095 -0.019" rpy="0 0 0" />
+      <origin xyz="-0.10998 -0.095 -0.0204" rpy="0 0 0" />
       <parent link="base_link" />
       <child link="MT_behind_right" />

File: src/agv_gazebo/xacro_agv/caster_up_left.xacro (robot description, xacro)
@@ -25,5 +25,5 @@
     </link>
     <joint name="MT_up_left_jt" type="fixed">
-      <origin xyz="0.11002 0.095 -0.019" rpy="0 0 0" />
+      <origin xyz="0.11002 0.095 -0.0204" rpy="0 0 0" />
       <parent link="base_link" />
       <child link="MT_up_left" />

File: src/agv_gazebo/xacro_agv/caster_up_right.xacro (robot description, xacro)
@@ -25,5 +25,5 @@
     </link>
     <joint name="MT_up_right_jt" type="fixed">
-      <origin xyz="0.11002 -0.095 -0.019" rpy="0 0 0" />
+      <origin xyz="0.11002 -0.095 -0.0204" rpy="0 0 0" />
       <parent link="base_link" />
       <child link="MT_up_right" />
